File: PCB/CubBELMonitor/CubBELMonitor.kicad_pcb (KiCad board)
At the start: 2 copper layers, 80 x 59 mm, 54 parts, among them J1 UM232R, J2 UM232R, P1 Power, P2 SHIFT, P20 Conn_01x02_Male, P21 Conn_01x02_Male, P3 GNSS, P30 Debug, P4 LED, P5 Debug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

Commit message: 基板更新
Parts:
- added R18: 1K, Resistor_SMD:R_0603_1608Metric_Pad1.05x0.95mm_HandSolder, F.Cu at (106.8, 75.0)
- C31, D10, J1, J2, P21, P30, Q31, Q32, R20, R21, R22, R31, R32, R33, R34: moved to B.Cu
- P20: moved to F.Cu
- moved J2 97.2 mm to (158.2, 105.9), turned to 0 degrees
- moved J1 80.9 mm to (143.0, 105.9), turned to 0 degrees
- moved R34 79.2 mm to (152.1, 95.1), turned to 90 degrees
- moved R33 76.3 mm to (149.0, 95.1), turned to 270 degrees
- moved Q32 75.6 mm to (153.1, 90.2), turned to 90 degrees
- moved R31 72.6 mm to (154.0, 85.9), turned to 180 degrees
- moved Q31 71.2 mm to (148.0, 90.2), turned to 90 degrees
- moved R32 69.1 mm to (149.7, 85.9), turned to 0 degrees
- moved D10 68.3 mm to (125.0, 34.4), turned to 90 degrees
- moved C31 67.7 mm to (154.1, 79.5), turned to 0 degrees
- moved P30 60.4 mm to (145.5, 75.4), turned to 270 degrees
- moved R20 59.7 mm to (126.4, 38.8), turned to 270 degrees
- moved R21 59.7 mm to (125.0, 38.8), turned to 270 degrees
- moved R22 59.7 mm to (123.6, 38.8), turned to 270 degrees
- moved P21 55.2 mm to (124.4, 41.1)
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Connections:
- C31 pad 1: Net-(C31-Pad1) -> /EN
- J1 pad 1: /TXD -> /ESP32<-PC
- J1 pad 5: /RXD -> /ESP32->PC
- P30 pad 1: /RXD -> /ESP32->PC
- P30 pad 2: /TXD -> /ESP32<-PC
- P30 pad 3: Net-(P30-Pad3) -> /IO0
- P30 pad 4: Net-(C31-Pad1) -> /EN
- P4 pad 1: Net-(P4-Pad1) -> Net-(D10-Pad4)
- P4 pad 2: Net-(P4-Pad2) -> Net-(P20-Pad2)
- P4 pad 3: Net-(P4-Pad3) -> Net-(P21-Pad1)
- P4 pad 4: Net-(P4-Pad4) -> Net-(P21-Pad2)
- Q31 pad 3: Net-(P30-Pad3) -> /IO0
- Q32 pad 3: Net-(C31-Pad1) -> /EN
- R15 pad 1: Net-(P4-Pad2) -> Net-(P20-Pad2)
- R16 pad 1: Net-(P4-Pad3) -> Net-(P21-Pad1)
- R17 pad 1: Net-(P4-Pad4) -> Net-(P21-Pad2)
- R31 pad 2: Net-(C31-Pad1) -> /EN
- R32 pad 2: Net-(P30-Pad3) -> /IO0
- R5 pad 2: /BATT -> Net-(R18-Pad2)
- R6 pad 1: /BATT -> Net-(R18-Pad2)
- TH2 pad 1: Net-(P4-Pad1) -> Net-(D10-Pad4)
Routing:
- net /ESP32<-PC: track 49.3 -> 101.6 mm
- net /ESP32->PC: track 46.8 -> 89.1 mm
- net /IO0: track 41.5 -> 76.5 mm
- net /EN: track 79.4 -> 112.4 mm
- net /TXD: track 32.6 -> 0.00 mm
- net Net-(P21-Pad1): track 3.77 -> 32.0 mm
- net Net-(P20-Pad2): track 3.69 -> 28.5 mm
- net Net-(P21-Pad2): track 3.64 -> 27.6 mm
- net /RXD: track 21.4 -> 0.00 mm
- net Net-(D10-Pad4): track 18.5 -> 39.8 mm
- net /BATT: track 38.2 -> 19.4 mm, vias 2 -> 0
- net Net-(R18-Pad2): track 0.00 -> 17.0 mm, vias 0 -> 2
- net Net-(P4-Pad2): track 15.8 -> 0.00 mm
- net Net-(P30-Pad3): track 15.3 -> 0.00 mm
- net Net-(C31-Pad1): track 13.5 -> 0.00 mm
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Other:
- board size 80 x 59 mm -> 100 x 77 mm
- board text added: "CubBLEMonitor 2021.3.30 @n_yosihisa"
