File: PCB/CubBELMonitor/CubBELMonitor.sch (KiCad schematic (older format))
At the start: 51 parts, among them J1 UM232R, J2 UM232R, P1 Power, P2 SHIFT, P20 LED, P3 GNSS, P30 Debug, P4 LED, P5 Debug, P6 IG, Q1 2SC3325, Q2 2SC3325, Q3 2SC3325, Q31 2SC2712, Q32 2SC2712, U1 ESP32-WROOM-32D, U2 LT1129IST-3.3

Commit message: ボード追加
Parts:
- removed P20: LED, symbol Connector_Generic:Conn_01x04
- added C3: 0.1u, Capacitor_SMD:C_0603_1608Metric_Pad1.05x0.95mm_HandSolder, symbol Device:C
- added P20, P21: Conn_01x02_Male, user_library:3mmLED_, symbol Connector:Conn_01x02_Male
- added TH4: microSMD010, Resistor_SMD:R_1210_3225Metric_Pad1.42x2.65mm_HandSolder, symbol Device:Thermistor_PTC
- C1: footprint (none) -> Capacitor_SMD:C_0603_1608Metric_Pad1.05x0.95mm_HandSolder
- C2, C31: footprint (none) -> Capacitor_SMD:C_0805_2012Metric_Pad1.15x1.40mm_HandSolder
- D1, D2, D3: footprint (none) -> Diode_SMD:D_SOD-123
- D10: footprint (none) -> LED_SMD:LED_Avago_PLCC6_3x2.8mm
- J1, J2: footprint (none) -> Connector_PinHeader_2.54mm:PinHeader_1x12_P2.54mm_Vertical
- P1: footprint (none) -> Connector_JST:JST_XH_S2B-XH-A_1x02_P2.50mm_Horizontal
- P2, P3, P4: footprint (none) -> Connector_JST:JST_XH_S4B-XH-A_1x04_P2.50mm_Horizontal
- P30: footprint (none) -> Connector_PinHeader_2.54mm:PinHeader_1x05_P2.54mm_Vertical
- P5: footprint (none) -> Connector_PinSocket_2.54mm:PinSocket_1x05_P2.54mm_Vertical
- P6: footprint (none) -> Connector_JST:JST_XH_B2B-XH-A_1x02_P2.50mm_Vertical
- Q1, Q2, Q3, Q31, Q32: footprint (none) -> Package_TO_SOT_SMD:SC-59
- R1, R10, R11, R12, R13, R14, R15, R16, R17, R2, R20, R21, R22, R3, R31, R32, R33, R34, R4, R5, R6, R7, R8, R9, TH1: footprint (none) -> Resistor_SMD:R_0603_1608Metric_Pad1.05x0.95mm_HandSolder
- TH2: value PTC -> microSMD010; footprint (none) -> Resistor_SMD:R_1210_3225Metric_Pad1.42x2.65mm_HandSolder; akizuki (none) -> P-01316
- TH3: value PTC -> SMD1812P125TS; footprint (none) -> Resistor_SMD:R_1812_4532Metric_Pad1.30x3.40mm_HandSolder; akizuki (none) -> P-10074
Connections:
- net +3V3: now also TH4.2; no longer P3.1 (Pin_1)
- net ESP32->GNSS: now also P3.3 (Pin_3); no longer P3.4 (Pin_4)
- net ESP32<-GNSS: now also P3.4 (Pin_4); no longer P3.3 (Pin_3)
- net GND: now also C3.2
- net at D3.2 (A), R2.2, R3.1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: now also C3.1
- net at R20.2: now also P21.1 (Pin_1)
- net at R22.2: now also P21.2 (Pin_2)
- net at R21.2: now also P20.2 (Pin_2)
- net at D10.4 (BA), D10.5 (GA), D10.6 (RA): now also P20.1 (Pin_1)
- new net: P3.1 (Pin_1), TH4.1
Other:
- moved on the sheet: D3, R3, R4, R5, R6, R7, TH1, U1

Commit message: 基板更新
Parts:
- added R18: 1K, Resistor_SMD:R_0603_1608Metric_Pad1.05x0.95mm_HandSolder, symbol Device:R
Connections:
- net RXD is gone; now on net ESP32->PC: J1.5 (Pin_5), P30.1 (Pin_1)
- net TXD is gone; now on net ESP32<-PC: J1.1 (Pin_1), P30.2 (Pin_2)
- net BATT: now also R18.1; no longer R5.2, R6.1
- net EN: now also C31.1, P30.4 (Pin_4), Q32.3 (C), R31.2
- net IO0: now also P30.3 (Pin_3), Q31.3 (C), R32.2
- net at P21.1 (Pin_1), R20.2: now also P4.3 (Pin_3), R16.1
- net at P21.2 (Pin_2), R22.2: now also P4.4 (Pin_4), R17.1
- net at P20.2 (Pin_2), R21.2: now also P4.2 (Pin_2), R15.1
- net at P4.1 (Pin_1), TH2.1: now also D10.4 (BA), D10.5 (GA), D10.6 (RA), P20.1 (Pin_1)
- new net: R18.2, R5.2, R6.1
Other:
- moved on the sheet: R7, TH1
Changed lines of the file:
@@
 Wire Wire Line
 	1850 3600 1850 3550
-Text Label 2100 3950 0    50   ~ 0
+Text Label 2500 3950 0    50   ~ 0
 BATT
 $Comp
@@
 $EndComp
 Wire Wire Line
-	2400 3600 2400 3550
-Wire Wire Line
-	2400 4450 2400 4400
-Text Label 2650 3950 0    50   ~ 0
+	2900 3600 2900 3550
+Wire Wire Line
+	2900 4450 2900 4400
+Text Label 3150 3950 0    50   ~ 0
 TEMP
 $Comp
 L power:+3.3V #PWR07
 U 1 1 60278E4B
-P 2400 3550
-F 0 "#PWR07" H 2400 3400 50  0001 C CNN
-F 1 "+3.3V" H 2415 3723 50  0000 C CNN
-F 2 "" H 2400 3550 50  0001 C CNN
-F 3 "" H 2400 3550 50  0001 C CNN
-	1    2400 3550
+P 2900 3550
+F 0 "#PWR07" H 2900 3400 50  0001 C CNN
+F 1 "+3.3V" H 2915 3723 50  0000 C CNN
+F 2 "" H 2900 3550 50  0001 C CNN
+F 3 "" H 2900 3550 50  0001 C CNN
+	1    2900 3550
 	1    0    0    -1
 $EndComp
@@
 L power:GND #PWR08
 U 1 1 6027843D
-P 2400 4450
-F 0 "#PWR08" H 2400 4200 50  0001 C CNN
-F 1 "GND" H 2405 4277 50  0000 C CNN
-F 2 "" H 2400 4450 50  0001 C CNN
-F 3 "" H 2400 4450 50  0001 C CNN
-	1    2400 4450
+P 2900 4450
+F 0 "#PWR08" H 2900 4200 50  0001 C CNN
+F 1 "GND" H 2905 4277 50  0000 C CNN
+F 2 "" H 2900 4450 50  0001 C CNN
+F 3 "" H 2900 4450 50  0001 C CNN
+	1    2900 4450
 	1    0    0    -1
 $EndComp
@@
 L Device:R R7
 U 1 1 60275875
-P 2400 3750
-F 0 "R7" H 2470 3796 50  0000 L CNN
-F 1 "10K" H 2470 3705 50  0000 L CNN
-F 2 "Resistor_SMD:R_0603_1608Metric_Pad1.05x0.95mm_HandSolder" V 2330 3750 50  0001 C CNN
-F 3 "~" H 2400 3750 50  0001 C CNN
-	1    2400 3750
+P 2900 3750
+F 0 "R7" H 2970 3796 50  0000 L CNN
+F 1 "10K" H 2970 3705 50  0000 L CNN
+F 2 "Resistor_SMD:R_0603_1608Metric_Pad1.05x0.95mm_HandSolder" V 2830 3750 50  0001 C CNN
+F 3 "~" H 2900 3750 50  0001 C CNN
+	1    2900 3750
 	1    0    0    -1
 $EndComp
@@
 L Device:Thermistor TH1
 U 1 1 602753ED
-P 2400 4200
-F 0 "TH1" H 2505 4246 50  0000 L CNN
-F 1 "Thermistor" H 2505 4155 50  0000 L CNN
-F 2 "Resistor_SMD:R_0603_1608Metric_Pad1.05x0.95mm_HandSolder" H 2400 4200 50  0001 C CNN
-F 3 "~" H 2400 4200 50  0001 C CNN
-	1    2400 4200
+P 2900 4200
+F 0 "TH1" H 3005 4246 50  0000 L CNN
+F 1 "Thermistor" H 3005 4155 50  0000 L CNN
+F 2 "Resistor_SMD:R_0603_1608Metric_Pad1.05x0.95mm_HandSolder" H 2900 4200 50  0001 C CNN
+F 3 "~" H 2900 4200 50  0001 C CNN
+	1    2900 4200
 	1    0    0    -1
 $EndComp
@@
 $EndComp
 Wire Wire Line
-	1850 3900 1850 3950
-Wire Wire Line
-	2400 3900 2400 3950
-Wire Wire Line
-	2100 3950 1850 3950
-Connection ~ 1850 3950
-Wire Wire Line
-	1850 3950 1850 4050
-Wire Wire Line
-	2650 3950 2400 3950
-Connection ~ 2400 3950
-Wire Wire Line
-	2400 3950 2400 4000
+	2900 3900 2900 3950
+Wire Wire Line
+	3150 3950 2900 3950
+Connection ~ 2900 3950
+Wire Wire Line
+	2900 3950 2900 4000
 $Comp
 L Connector_Generic:Conn_01x02 P6
@@
 Wire Wire Line
 	7650 1750 7650 1600
-Wire Wire Line
-	7650 1600 7900 1600
-Wire Wire Line
-	7900 1500 7450 1500
 Wire Wire Line
 	7450 1500 7450 1750
@@
 	6500 2450 6600 2450
 Wire Wire Line
-	7400 1400 7900 1400
-Wire Wire Line
 	6700 1400 7100 1400
 $Comp
@@
 Wire Wire Line
 	10500 1400 10500 1650
-Wire Wire Line
-	9250 1400 10500 1400
 $Comp
 L Device:LED_RGB D10
@@
 $EndComp
 Wire Wire Line
-	9250 1750 9450 1750
+	9250 1750 9350 1750
 Wire Wire Line
 	9450 1750 9450 2050
-Wire Wire Line
-	9250 1650 9650 1650
-Wire Wire Line
-	9250 1500 9550 1500
 Wire Wire Line
 	9550 1500 9550 1850
@@
 Wire Wire Line
 	2400 3000 2400 2900
+$Comp
+L Device:R R18
+U 1 1 60608949
+P 2150 3950
+F 0 "R18" H 2220 3996 50  0000 L CNN
+F 1 "1K" H 2220 3905 50  0000 L CNN
+F 2 "Resistor_SMD:R_0603_1608Metric_Pad1.05x0.95mm_HandSolder" V 2080 3950 50  0001 C CNN
+F 3 "~" H 2150 3950 50  0001 C CNN
+	1    2150 3950
+	0    1    1    0
+$EndComp
+Wire Wire Line
+	1850 3900 1850 3950
+Wire Wire Line
+	2000 3950 1850 3950
+Connection ~ 1850 3950
+Wire Wire Line
+	1850 3950 1850 4050
+Wire Wire Line
+	2300 3950 2500 3950
+Text Label 8250 5250 2    50   ~ 0
+ESP32<-PC
+Text Label 8250 5150 2    50   ~ 0
+ESP32->PC
+Text Label 8250 5450 2    50   ~ 0
+EN
+Text Label 8250 5350 2    50   ~ 0
+IO0
+Wire Wire Line
+	7650 1600 7850 1600
+Wire Wire Line
+	9250 1650 9350 1650
+Wire Wire Line
+	9250 1500 9350 1500
+Wire Wire Line
+	7900 1500 7850 1500
+Wire Wire Line
+	9250 1400 9350 1400
+Wire Wire Line
+	7400 1400 7850 1400
+Wire Wire Line
+	7850 1700 7850 1650
+Wire Wire Line
+	7850 1650 8750 1650
+Wire Wire Line
+	8750 1650 8750 1700
+Wire Wire Line
+	8750 1700 9350 1700
+Wire Wire Line
+	9350 1700 9350 1750
+Connection ~ 7850 1700
+Connection ~ 9350 1750
+Wire Wire Line
+	9350 1750 9450 1750
+Wire Wire Line
+	9350 1650 9350 1550
+Wire Wire Line
+	9350 1550 7850 1550
+Wire Wire Line
+	7850 1550 7850 1600
+Connection ~ 9350 1650
+Wire Wire Line
+	9350 1650 9650 1650
+Connection ~ 7850 1600
+Wire Wire Line
+	7850 1600 7900 1600
+Wire Wire Line
+	7850 1500 7850 1450
+Wire Wire Line
+	7850 1450 9350 1450
+Wire Wire Line
+	9350 1450 9350 1500
+Connection ~ 7850 1500
+Wire Wire Line
+	7850 1500 7450 1500
+Connection ~ 9350 1500
+Wire Wire Line
+	9350 1500 9550 1500
+Wire Wire Line
+	9350 1400 9350 1350
+Wire Wire Line
+	9350 1350 7850 1350
+Wire Wire Line
+	7850 1350 7850 1400
+Connection ~ 9350 1400
+Wire Wire Line
+	9350 1400 10500 1400
+Connection ~ 7850 1400
+Wire Wire Line
+	7850 1400 7900 1400
 $EndSCHEMATC
